Commit message: Finished designing 3-link, 2-joint robot

File: body.urdf (robot description, URDF)
Before this commit: robot robot, 7 links, 6 joints
Links:
- removed link Link3
- removed link Link4
- removed link Link5
- removed link Link6
Joints:
- removed joint Link2_Link3
- removed joint Link3_Link4
- removed joint Link4_Link5
- removed joint Link5_Link6
- joint Link0_Link1: origin xyz=0 0 1 rpy=0 0 0 -> xyz=0.5 0 1 rpy=0 0 0
- joint Link1_Link2: origin xyz=0 0 1 rpy=0 0 0 -> xyz=1 0 0 rpy=0 0 0

Commit message: Successful closed-loop control of robot!

File: body.urdf (robot description, URDF)
Before this commit: robot robot, 3 links, 2 joints
Joints:
- joint Torso_BackLeg: origin xyz=-0.5 0 1 rpy=0 0 0 -> xyz=-0.5 0 1.0 rpy=0 0 0
- joint Torso_FrontLeg: origin xyz=0.5 0 1 rpy=0 0 0 -> xyz=0.5 0 1.0 rpy=0 0 0

Commit message: Progress for now!

File: body.urdf (robot description, URDF)
Before this commit: robot robot, 3 links, 2 joints
Links:
- link BackLeg: geometry collision box size=0.2 1 0.2; visual box size=0.2 1 0.2
- link FrontLeg: geometry collision box size=0.2 1 0.2; visual box size=0.2 1 0.2
Joints:
- joint Torso_BackLeg: origin xyz=-0.5 0 1.0 rpy=0 0 0 -> xyz=0 0.5 1 rpy=0 0 0
- joint Torso_FrontLeg: origin xyz=0.5 0 1.0 rpy=0 0 0 -> xyz=0 -0.5 1 rpy=0 0 0

Commit message: Quadruped

File: body.urdf (robot description, URDF)
Before this commit: robot robot, 3 links, 2 joints
Links:
- added link BackLower, mass 1; collision box size=0.2 0.2 1; visual box size=0.2 0.2 1
- added link FrontLower, mass 1; collision box size=0.2 0.2 1; visual box size=0.2 0.2 1
- added link LeftLeg, mass 1; collision box size=1 0.2 0.2; visual box size=1 0.2 0.2
- added link LeftLower, mass 1; collision box size=0.2 0.2 1; visual box size=0.2 0.2 1
- added link RightLeg, mass 1; collision box size=1 0.2 0.2; visual box size=1 0.2 0.2
- added link RightLower, mass 1; collision box size=0.2 0.2 1; visual box size=0.2 0.2 1
Joints:
- added joint BackLeg_BackLower: type revolute, parent BackLeg, child BackLower, origin xyz=0 -1 0 rpy=0 0 0, axis 1 0 1, limit lower=-3.14159 upper=3.14159 effort=0.0 velocity=0.0
- added joint FrontLeg_FrontLower: type revolute, parent FrontLeg, child FrontLower, origin xyz=0 1 0 rpy=0 0 0, axis 1 0 1, limit lower=-3.14159 upper=3.14159 effort=0.0 velocity=0.0
- added joint LeftLeg_LeftLower: type revolute, parent LeftLeg, child LeftLower, origin xyz=-1 0 0 rpy=0 0 0, axis 0 1 1, limit lower=-3.14159 upper=3.14159 effort=0.0 velocity=0.0
- added joint RightLeg_RightLower: type revolute, parent RightLeg, child RightLower, origin xyz=1 0 0 rpy=0 0 0, axis 0 1 1, limit lower=-3.14159 upper=3.14159 effort=0.0 velocity=0.0
- added joint Torso_LeftLeg: type revolute, parent Torso, child LeftLeg, origin xyz=-0.5 0 1 rpy=0 0 0, axis 0 1 1, limit lower=-3.14159 upper=3.14159 effort=0.0 velocity=0.0
- added joint Torso_RightLeg: type revolute, parent Torso, child RightLeg, origin xyz=0.5 0 1 rpy=0 0 0, axis 0 1 1, limit lower=-3.14159 upper=3.14159 effort=0.0 velocity=0.0
- joint Torso_BackLeg: axis 0 1 0 -> 1 0 1; origin xyz=0 0.5 1 rpy=0 0 0 -> xyz=0 -0.5 1 rpy=0 0 0
- joint Torso_FrontLeg: axis 0 1 0 -> 1 0 1; origin xyz=0 -0.5 1 rpy=0 0 0 -> xyz=0 0.5 1 rpy=0 0 0

Commit message: Successful build of capsule leg robot!

File: body.urdf (robot description, URDF)
Before this commit: robot robot, 9 links, 8 joints
Links:
- link BackLeg: geometry collision capsule length=1 radius=0.2; visual capsule length=1 radius=0.2
- link BackLower: geometry collision capsule length=1 radius=0.2; visual capsule length=1 radius=0.2
- link FrontLeg: geometry collision capsule length=1 radius=0.2; visual capsule length=1 radius=0.2
- link FrontLower: geometry collision capsule length=1 radius=0.2; visual capsule length=1 radius=0.2
- link LeftLeg: geometry collision capsule length=1 radius=0.2; visual capsule length=1 radius=0.2
- link LeftLower: geometry collision capsule length=1 radius=0.2; visual capsule length=1 radius=0.2
- link RightLeg: geometry collision capsule length=1 radius=0.2; visual capsule length=1 radius=0.2
- link RightLower: geometry collision capsule length=1 radius=0.2; visual capsule length=1 radius=0.2
Joints:
- joint Torso_BackLeg: origin xyz=0 -0.5 1 rpy=0 0 0 -> xyz=0 -0.5 1.2 rpy=0 0 0
- joint Torso_FrontLeg: origin xyz=0 0.5 1 rpy=0 0 0 -> xyz=0 0.5 1.2 rpy=0 0 0
- joint Torso_LeftLeg: origin xyz=-0.5 0 1 rpy=0 0 0 -> xyz=-0.5 0 1.2 rpy=0 0 0
- joint Torso_RightLeg: origin xyz=0.5 0 1 rpy=0 0 0 -> xyz=0.5 0 1.2 rpy=0 0 0
